Commit message: variable friction hand controllers

File: gripper/urdf/gripper.urdf (robot description, URDF)
Before this commit: robot gripper, 4 links, 3 joints
Joints:
- joint J1: limit lower=0 upper=0 effort=0 velocity=0 -> lower=0 upper=0 effort=1 velocity=0.5; type revolute -> continuous
- joint J2: limit lower=0 upper=0 effort=0 velocity=0 -> lower=0 upper=0 effort=1 velocity=0.5; type revolute -> continuous
