Commit message: collision changes

File: franka_description/robots/hand.xacro (robot description, xacro)
@@ -35,5 +35,9 @@
           <mesh filename="package://franka_description/meshes/collision/finger.stl"/>
         </geometry>
-        <surface>
+        <contact_coefficients
+          mu="0.5"
+          kp="1000000"
+          kd="10"/>
+        <!-- <surface>
           <friction>
             <ode>
@@ -45,5 +49,5 @@
             </torsional>
           </friction>
-        </surface>
+        </surface> -->
       </collision>
 	<inertial>
@@ -64,5 +68,9 @@
           <mesh filename="package://franka_description/meshes/collision/finger.stl"/>
         </geometry>
-        <surface>
+        <contact_coefficients
+          mu="0.5"
+          kp="1000000"
+          kd="10"/>
+        <!-- <surface>
           <friction>
             <ode>
@@ -74,5 +82,5 @@
             </torsional>
           </friction>
-        </surface>
+        </surface> -->
       </collision>
 	<inertial>

File: object_description/urdf/table.urdf (robot description, URDF)
Before this commit: robot block_object, 1 links, 0 joints
Links:
- removed link block
- added link table, mass 0.5; collision box size=0.5 0.5 0.3; visual box size=0.5 0.5 0.3

Commit message: gripper controllers and testing

File: franka_description/robots/hand.xacro (robot description, xacro)
@@ -37,6 +37,6 @@
         <contact_coefficients
           mu="0.5"
-          kp="1000000"
-          kd="10"/>
+          kp="100"
+          kd="1"/>
         <!-- <surface>
           <friction>
@@ -70,6 +70,6 @@
         <contact_coefficients
           mu="0.5"
-          kp="1000000"
-          kd="10"/>
+          kp="100"
+          kd="1"/>
         <!-- <surface>
           <friction>

File: gripper/urdf/gripper.urdf (robot description, URDF)
Before this commit: robot gripper, 4 links, 3 joints
Joints:
- joint J1: limit lower=0 upper=0 effort=1 velocity=0.5 -> lower=0 upper=0 effort=10 velocity=0.5
- joint J2: limit lower=0 upper=0 effort=1 velocity=0.5 -> lower=0 upper=0 effort=10 velocity=0.5

File: object_description/urdf/long_block.urdf (robot description, URDF)
Before this commit: robot block_object, 1 links, 0 joints
Links:
- link block: geometry collision box size=0.03 0.03 0.1; visual box size=0.03 0.03 0.1
